File: Panelize - Xonik Noise A6 w.logo v2.0.sch (EAGLE design)
At the start: 38 parts, among them IC1 TL074D, T1 NOISE-2N3904

Commit message: Changed recommended external trimmer for 50k to 100k to be able to reach a high enough amplitude
Other:
- note added: "Mount EITHER 20k or external 50k trimmer NB: 2.43k in simulation???"
- note removed: "Use external 100k trimmer for good amplitude adjustability NB: 2.43k in simulation???"
Changed lines of the file:
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@@
 <sheet>
 <plain>
-<text x="66.04" y="139.7" size="1.778" layer="97">Use external 100k trimmer
-for good amplitude adjustability
+<text x="66.04" y="139.7" size="1.778" layer="97">Mount EITHER 20k or external 50k trimmer
 NB: 2.43k in simulation???</text>
 <text x="139.7" y="73.66" size="1.778" layer="97">Approximated
