File: Xonik Noise A6 w.logo v2.1-12v.sch (EAGLE design)
At the start: 38 parts, among them IC1 TL074D, T1 NOISE-2N3904

Commit message: Working on 12v version with 0603 res
Parts:
- 1, 10, 11, 12, 13, 14, 15, 16, 17, 2, 3, 4, 5, 6, 7, 8, 9: device resistor:R-EU_R0805 -> rcl:R-EU_R0603
- C1, C2, C3, C4, C5, C6, C7, C8, C9: device resistor:C-EUC0805 -> rcl:C-EUC0603
- C10: device resistor:C-EUC0603 -> rcl:C-EUC0603
Connections:
- net +15V renamed +12V
- net -15V renamed -12V

Commit message: Version 2.1 12V completed I think
Parts:
- removed NOISE_IN: (no value), joakim:MA01-1JP
- IC1: value TL074D -> TL074JT; device linear:TL074D -> joakim:TL074JT
Connections:
- net GND: now also IC1B.-IN; no longer IC1B.+IN
- net N$1: now also IC1A.+IN; no longer IC1A.-IN
- net N$10: now also IC1D.-IN; no longer IC1D.+IN
- net N$12: now also IC1C.-IN; no longer IC1C.+IN
- net N$17: now also IC1B.+IN; no longer IC1B.-IN
- net N$2: now also IC1D.+IN; no longer IC1D.-IN
- net N$3: now also IC1C.+IN; no longer IC1C.-IN
- net N$7: no longer NOISE_IN.1
- net N$8: now also IC1A.-IN; no longer IC1A.+IN
Changed lines of the file:
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@@
 <layer number="54" name="bGND_GNDA" color="1" fill="9" visible="no" active="no"/>
 <layer number="56" name="wert" color="7" fill="1" visible="no" active="no"/>
+<layer number="57" name="tCAD" color="7" fill="1" visible="no" active="no"/>
+<layer number="59" name="tCarbon" color="7" fill="1" visible="no" active="no"/>
+<layer number="60" name="bCarbon" color="7" fill="1" visible="no" active="no"/>
+<layer number="88" name="SimResults" color="9" fill="1" visible="yes" active="yes"/>
+<layer number="89" name="SimProbes" color="9" fill="1" visible="yes" active="yes"/>
 <layer number="90" name="Modules" color="5" fill="1" visible="yes" active="yes"/>
 <layer number="91" name="Nets" color="2" fill="1" visible="yes" active="yes"/>
@@
 <layer number="126" name="BIFRNTMAT" color="7" fill="1" visible="yes" active="yes"/>
 <layer number="127" name="Info2" color="7" fill="1" visible="yes" active="yes"/>
+<layer number="128" name="_bValues" color="7" fill="1" visible="no" active="yes"/>
+<layer number="129" name="Mask" color="7" fill="1" visible="yes" active="yes"/>
 <layer number="130" name="SMDSTROOK" color="7" fill="1" visible="yes" active="yes"/>
 <layer number="131" name="tAdjust" color="7" fill="1" visible="yes" active="yes"/>
@@
 <layer number="136" name="BGA_DED" color="14" fill="1" visible="yes" active="yes"/>
 <layer number="144" name="Drill_legend" color="7" fill="1" visible="yes" active="yes"/>
+<layer number="150" name="Notes" color="7" fill="1" visible="no" active="yes"/>
 <layer number="151" name="HeatSink" color="7" fill="1" visible="yes" active="yes"/>
+<layer number="152" name="_bDocu" color="7" fill="1" visible="no" active="yes"/>
+<layer number="153" name="FabDoc1" color="7" fill="1" visible="no" active="yes"/>
+<layer number="154" name="FabDoc2" color="7" fill="1" visible="no" active="yes"/>
+<layer number="155" name="FabDoc3" color="7" fill="1" visible="no" active="yes"/>
 <layer number="199" name="Contour" color="7" fill="1" visible="yes" active="yes"/>
 <layer number="200" name="200bmp" color="1" fill="10" visible="no" active="no"/>
@@
 <layer number="215" name="215bmp" color="7" fill="1" visible="yes" active="yes"/>
 <layer number="216" name="BottomExtra" color="7" fill="1" visible="yes" active="yes"/>
+<layer number="217" name="217bmp" color="18" fill="1" visible="no" active="no"/>
+<layer number="218" name="218bmp" color="19" fill="1" visible="no" active="no"/>
+<layer number="219" name="219bmp" color="20" fill="1" visible="no" active="no"/>
+<layer number="220" name="220bmp" color="21" fill="1" visible="no" active="no"/>
+<layer number="221" name="221bmp" color="22" fill="1" visible="no" active="no"/>
+<layer number="222" name="222bmp" color="23" fill="1" visible="no" active="no"/>
+<layer number="223" name="223bmp" color="24" fill="1" visible="no" active="no"/>
+<layer number="224" name="224bmp" color="25" fill="1" visible="no" active="no"/>
+<layer number="225" name="225bmp" color="7" fill="1" visible="yes" active="yes"/>
+<layer number="226" name="226bmp" color="7" fill="1" visible="yes" active="yes"/>
+<layer number="227" name="227bmp" color="7" fill="1" visible="yes" active="yes"/>
+<layer number="228" name="228bmp" color="7" fill="1" visible="yes" active="yes"/>
+<layer number="229" name="229bmp" color="7" fill="1" visible="yes" active="yes"/>
+<layer number="230" name="230bmp" color="7" fill="1" visible="yes" active="yes"/>
+<layer number="231" name="Eagle3D_PG1" color="7" fill="1" visible="no" active="no"/>
+<layer number="232" name="Eagle3D_PG2" color="7" fill="1" visible="no" active="no"/>
+<layer number="233" name="Eagle3D_PG3" color="7" fill="1" visible="no" active="no"/>
+<layer number="248" name="Housing" color="7" fill="1" visible="no" active="yes"/>
+<layer number="249" name="Edge" color="7" fill="1" visible="no" active="yes"/>
 <layer number="250" name="Descript" color="7" fill="1" visible="no" active="no"/>
 <layer number="251" name="SMDround" color="7" fill="1" visible="no" active="no"/>
@@
 <part name="C8" library="rcl" library_urn="urn:adsk.eagle:library:334" deviceset="C-EU" device="C0603" package3d_urn="urn:adsk.eagle:package:23616/2" value="220n"/>
 <part name="C9" library="rcl" library_urn="urn:adsk.eagle:library:334" deviceset="C-EU" device="C0603" package3d_urn="urn:adsk.eagle:package:23616/2" value="2n2"/>
-<part name="IC1" library="linear" deviceset="TL074" device="D"/>
+<part name="IC1" library="joakim" deviceset="TL074J" device="T"/>
 <part name="C10" library="rcl" library_urn="urn:adsk.eagle:library:334" deviceset="C-EU" device="C0603" package3d_urn="urn:adsk.eagle:package:23616/2" value="100nF"/>
-<part name="NOISE_IN" library="joakim" deviceset="MA01-1J" device="P"/>
 <part name="LEVEL1" library="joakim" deviceset="MA01-1J" device="P"/>
 <part name="LEVEL2" library="joakim" deviceset="MA01-1J" device="P"/>
@@
 <attribute name="VALUE" x="26.416" y="37.719" size="1.778" layer="96" rot="R180"/>
 </instance>
-<instance part="NOISE_IN" gate="G$1" x="60.96" y="93.98" smashed="yes" rot="R90">
-<attribute name="VALUE" x="66.04" y="92.71" size="1.778" layer="96" rot="R90"/>
-<attribute name="NAME" x="57.658" y="92.71" size="1.778" layer="95" rot="R90"/>
-</instance>
 <instance part="LEVEL1" gate="G$1" x="86.36" y="134.62" smashed="yes" rot="R270">
 <attribute name="VALUE" x="81.28" y="135.89" size="1.778" layer="96" rot="R270"/>
@@
 <segment>
 <pinref part="2" gate="G$1" pin="1"/>
-<pinref part="IC1" gate="A" pin="-IN"/>
+<pinref part="IC1" gate="A" pin="+IN"/>
 <wire x1="86.36" y1="111.76" x2="86.36" y2="119.38" width="0.1524" layer="91"/>
 <pinref part="LEVEL1" gate="G$1" pin="1"/>
@@
 <pinref part="5" gate="G$1" pin="2"/>
 <pinref part="6" gate="G$1" pin="1"/>
-<pinref part="IC1" gate="D" pin="-IN"/>
+<pinref part="IC1" gate="D" pin="+IN"/>
 <wire x1="119.38" y1="111.76" x2="119.38" y2="119.38" width="0.1524" layer="91"/>
 <junction x="119.38" y="119.38"/>
@@
 <pinref part="13" gate="G$1" pin="2"/>
 <pinref part="14" gate="G$1" pin="1"/>
-<pinref part="IC1" gate="C" pin="-IN"/>
+<pinref part="IC1" gate="C" pin="+IN"/>
 <wire x1="119.38" y1="68.58" x2="119.38" y2="76.2" width="0.1524" layer="91"/>
 <junction x="119.38" y="76.2"/>
@@
 </segment>
 <segment>
-<pinref part="IC1" gate="B" pin="+IN"/>
+<pinref part="IC1" gate="B" pin="-IN"/>
 <pinref part="GND8" gate="1" pin="GND"/>
 </segment>
@@
 <segment>
 <pinref part="1" gate="G$1" pin="1"/>
-<pinref part="NOISE_IN" gate="G$1" pin="1"/>
 <pinref part="C1" gate="G$1" pin="1"/>
-<wire x1="60.96" y1="106.68" x2="60.96" y2="101.6" width="0.1524" layer="91"/>
 <wire x1="73.66" y1="106.68" x2="60.96" y2="106.68" width="0.1524" layer="91"/>
 <junction x="60.96" y="106.68"/>
@@
 <pinref part="4" gate="G$1" pin="1"/>
 <wire x1="81.28" y1="106.68" x2="83.82" y2="106.68" width="0.1524" layer="91"/>
-<pinref part="IC1" gate="A" pin="+IN"/>
+<pinref part="IC1" gate="A" pin="-IN"/>
 <wire x1="83.82" y1="106.68" x2="86.36" y2="106.68" width="0.1524" layer="91"/>
 <junction x="83.82" y="106.68"/>
@@
 <segment>
 <pinref part="C2" gate="G$1" pin="2"/>
-<pinref part="IC1" gate="D" pin="+IN"/>
+<pinref part="IC1" gate="D" pin="-IN"/>
 <wire x1="114.3" y1="106.68" x2="116.84" y2="106.68" width="0.1524" layer="91"/>
 <pinref part="7" gate="G$1" pin="2"/>
@@
 <junction x="109.22" y="63.5"/>
 <junction x="119.38" y="63.5"/>
-<pinref part="IC1" gate="C" pin="+IN"/>
+<pinref part="IC1" gate="C" pin="-IN"/>
 </segment>
 </net>
@@
 <segment>
 <pinref part="17" gate="G$1" pin="2"/>
-<pinref part="IC1" gate="B" pin="-IN"/>
+<pinref part="IC1" gate="B" pin="+IN"/>
 <wire x1="119.38" y1="17.78" x2="119.38" y2="27.94" width="0.1524" layer="91"/>
 <pinref part="C9" gate="G$1" pin="2"/>
