File: Xonik Noise A6 w.logo v2.1-12v.brd (EAGLE design)
At the start: 29.8 x 26 mm, 39 parts, among them IC1 TL074D, T1 NOISE-2N3904

Commit message: Version 2.1 12V completed I think
Parts:
- removed NOISE_IN: (no value), joakim:SIP-PIN01-1J
- IC1: value TL074D -> TL074JT; device linear:SO14 -> joakim:TSSOP14J
- moved 4 11.0 mm to (3.49, 11.3), turned to 270 degrees
- moved C1 9.87 mm to (1.27, 11.3)
- moved 1 9.51 mm to (3.49, 15.6), turned to 270 degrees
- moved C7 9.25 mm to (19.1, 19.7)
- moved 12 8.94 mm to (16.8, 19.7)
- moved C8 8.89 mm to (19.1, 6.99)
- moved GND 8.89 mm to (19.1, 3.17)
- moved LEVEL2 8.89 mm to (1.27, 3.17)
- moved PINK_OUT 8.89 mm to (8.89, 3.17)
- moved RED_OUT 8.89 mm to (11.4, 3.17)
- moved WHITE_OUT 8.89 mm to (6.35, 3.17)
- moved +15V 8.89 mm to (14.0, 3.17)
- moved LEVEL1 8.89 mm to (3.81, 3.17)
- moved -15V 8.89 mm to (16.5, 3.17)
- moved 9 8.87 mm to (19.2, 15.6)
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Connections:
- net GND: now also IC1.6; no longer IC1.5
- net N$1: now also IC1.3; no longer IC1.2
- net N$10: now also IC1.13; no longer IC1.12
- net N$12: now also IC1.9; no longer IC1.10
- net N$17: now also IC1.5; no longer IC1.6
- net N$2: now also IC1.12; no longer IC1.13
- net N$3: now also IC1.10; no longer IC1.9
- net N$7: no longer NOISE_IN.1
- net N$8: now also IC1.2; no longer IC1.3
Routing:
- net GND: track 123.7 -> 84.5 mm, vias 8 -> 9
- net N$8: track 23.4 -> 8.73 mm
- net N$12: track 44.4 -> 31.4 mm
- net +12V: track 33.3 -> 23.8 mm, vias 3 -> 1
- net N$16: track 18.6 -> 11.5 mm
- net N$13: track 9.93 -> 3.96 mm
- net N$7: track 9.92 -> 14.5 mm, vias 0 -> 2
- net -12V: track 24.5 -> 20.3 mm
- net N$17: track 15.9 -> 12.2 mm
- net N$9: track 23.8 -> 20.2 mm
- net N$10: track 21.5 -> 18.4 mm, vias 0 -> 2
- net N$3: track 16.2 -> 13.2 mm
- net N$18: track 14.7 -> 16.8 mm
- net N$14: track 29.7 -> 27.8 mm
- net N$2: track 13.0 -> 11.2 mm
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Other:
- board size 29.8 x 26 mm -> 20.3 x 22.9 mm
- board text added: "+12V"
- board text added: "-12V"
- board text added: "Trim"
- board text added: "v2.1 12V"
- board text removed: "+15V"
- board text removed: "-15V"
- board text removed: "1"
- board text removed: "10"
- board text removed: "11"
- board text removed: "12"
- board text removed: "13"
- board text removed: "14"
- board text removed: "15"
- board text removed: "16"
- board text removed: "17"
- board text removed: "2"
- board text removed: "3"
- board text removed: "4"
- board text removed: "5"
- board text removed: "50k Trim"
- board text removed: "6"
- board text removed: "7"
- board text removed: "8"
- board text removed: "9"
- board text removed: "C1"
- board text removed: "C2"
- board text removed: "C3"
- board text removed: "C4"
- board text removed: "C5"
- board text removed: "C6"
- board text removed: "C7"
- board text removed: "C8"
- board text removed: "C9"
- board text removed: "In"
- board text removed: "v2.0"

Commit message: Tiny tweaks
Other:
- board size 20.3 x 22.9 mm -> 20.3 x 22.7 mm
Changed lines of the file:
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@@
 <setting verticaltext="up"/>
 </settings>
-<grid distance="6.25" unitdist="mil" unit="mil" style="dots" multiple="1" display="yes" altdistance="0.025" altunitdist="inch" altunit="inch"/>
+<grid distance="6.25" unitdist="mil" unit="mm" style="dots" multiple="1" display="yes" altdistance="0.025" altunitdist="inch" altunit="inch"/>
 <layers>
 <layer number="1" name="Top" color="4" fill="1" visible="yes" active="yes"/>
@@
 <layer number="14" name="Route14" color="1" fill="6" visible="no" active="no"/>
 <layer number="15" name="Route15" color="4" fill="6" visible="no" active="no"/>
-<layer number="16" name="Bottom" color="1" fill="1" visible="no" active="yes"/>
+<layer number="16" name="Bottom" color="1" fill="1" visible="yes" active="yes"/>
 <layer number="17" name="Pads" color="2" fill="1" visible="yes" active="yes"/>
 <layer number="18" name="Vias" color="2" fill="1" visible="yes" active="yes"/>
 <layer number="19" name="Unrouted" color="6" fill="1" visible="yes" active="yes"/>
 <layer number="20" name="Dimension" color="15" fill="1" visible="yes" active="yes"/>
-<layer number="21" name="tPlace" color="7" fill="1" visible="no" active="yes"/>
+<layer number="21" name="tPlace" color="7" fill="1" visible="yes" active="yes"/>
 <layer number="22" name="bPlace" color="7" fill="1" visible="yes" active="yes"/>
-<layer number="23" name="tOrigins" color="15" fill="1" visible="no" active="yes"/>
+<layer number="23" name="tOrigins" color="15" fill="1" visible="yes" active="yes"/>
 <layer number="24" name="bOrigins" color="15" fill="1" visible="yes" active="yes"/>
-<layer number="25" name="tNames" color="7" fill="1" visible="no" active="yes"/>
+<layer number="25" name="tNames" color="7" fill="1" visible="yes" active="yes"/>
 <layer number="26" name="bNames" color="7" fill="1" visible="yes" active="yes"/>
 <layer number="27" name="tValues" color="7" fill="1" visible="no" active="yes"/>
@@
 <layer number="37" name="tTest" color="7" fill="1" visible="no" active="yes"/>
 <layer number="38" name="bTest" color="7" fill="1" visible="no" active="yes"/>
-<layer number="39" name="tKeepout" color="4" fill="11" visible="no" active="yes"/>
+<layer number="39" name="tKeepout" color="4" fill="11" visible="yes" active="yes"/>
 <layer number="40" name="bKeepout" color="1" fill="11" visible="yes" active="yes"/>
-<layer number="41" name="tRestrict" color="4" fill="10" visible="no" active="yes"/>
+<layer number="41" name="tRestrict" color="4" fill="10" visible="yes" active="yes"/>
 <layer number="42" name="bRestrict" color="1" fill="10" visible="yes" active="yes"/>
 <layer number="43" name="vRestrict" color="2" fill="10" visible="no" active="yes"/>
@@
 <layer number="49" name="Reference" color="7" fill="1" visible="no" active="yes"/>
 <layer number="50" name="dxf" color="7" fill="1" visible="no" active="no"/>
-<layer number="51" name="tDocu" color="7" fill="1" visible="no" active="yes"/>
+<layer number="51" name="tDocu" color="7" fill="1" visible="yes" active="yes"/>
 <layer number="52" name="bDocu" color="7" fill="1" visible="yes" active="yes"/>
 <layer number="53" name="tGND_GNDA" color="7" fill="9" visible="no" active="no"/>
@@
 <plain>
 <wire x1="0" y1="0" x2="20.32" y2="0" width="0" layer="20"/>
-<wire x1="20.32" y1="0" x2="20.32" y2="22.86" width="0" layer="20"/>
-<wire x1="20.32" y1="22.86" x2="0" y2="22.86" width="0" layer="20"/>
-<wire x1="0" y1="22.86" x2="0" y2="0" width="0" layer="20"/>
+<wire x1="20.32" y1="0" x2="20.32" y2="22.70125" width="0" layer="20"/>
+<wire x1="20.32" y1="22.70125" x2="0" y2="22.70125" width="0" layer="20"/>
+<wire x1="0" y1="22.70125" x2="0" y2="0" width="0" layer="20"/>
 <text x="3.01625" y="8.89" size="1.016" layer="26" rot="MR0">Trim</text>
 <text x="5.87375" y="5.23875" size="1.016" layer="26" rot="MR90">White</text>
@@
 <text x="19.1516" y="11.5951" size="1.778" layer="26" font="vector" rot="MR0">Triple noise</text>
 <text x="10.7442" y="16.1925" size="1.016" layer="25" font="vector">4V&amp;B</text>
-<text x="10.4775" y="8.89" size="1.016" layer="25">v2.1
+<text x="10.795" y="8.89" size="1.016" layer="25">v2.1
 12V</text>
 <polygon width="0.254" layer="26">
-<vertex x="0.3175" y="22.5425"/>
-<vertex x="0.3175" y="16.8275"/>
-<vertex x="6.0325" y="22.5425"/>
+<vertex x="0.3175" y="22.38375"/>
+<vertex x="0.3175" y="17.78"/>
+<vertex x="4.92125" y="22.38375"/>
 </polygon>
 <text x="2.7305" y="4.5085" size="1.016" layer="25">T1</text>
@@
 <contactref element="14" pad="2"/>
 <contactref element="15" pad="1"/>
-<wire x1="12.7" y1="16.1925" x2="12.065" y2="15.5575" width="0.3048" layer="1"/>
+<wire x1="12.7" y1="16.1925" x2="11.7475" y2="15.24" width="0.3048" layer="1"/>
 <wire x1="12.3825" y1="18.835" x2="12.7" y2="18.5175" width="0.3048" layer="1"/>
 <wire x1="12.7" y1="18.5175" x2="12.7" y2="16.1925" width="0.3048" layer="1"/>
 <wire x1="16.8275" y1="7.835" x2="16.8275" y2="8.5725" width="0.3048" layer="1"/>
-<wire x1="11.43" y1="14.9225" x2="12.065" y2="15.5575" width="0.3048" layer="16"/>
-<via x="12.065" y="15.5575" extent="1-16" drill="0.3302"/>
+<wire x1="11.43" y1="14.9225" x2="11.7475" y2="15.24" width="0.3048" layer="16"/>
+<via x="11.7475" y="15.24" extent="1-16" drill="0.3302"/>
 <wire x1="11.43" y1="5.715" x2="8.89" y2="3.175" width="0.3048" layer="16"/>
 <wire x1="11.43" y1="10.795" x2="11.43" y2="14.9225" width="0.3048" layer="16"/>
@@
 <wire x1="9.57" y1="15.5125" x2="9.8425" y2="15.24" width="0.3048" layer="1"/>
 <wire x1="9.8425" y1="15.24" x2="11.7475" y2="15.24" width="0.3048" layer="1"/>
-<wire x1="11.7475" y1="15.24" x2="12.065" y2="15.5575" width="0.3048" layer="1"/>
 <wire x1="16.8275" y1="8.5725" x2="16.51" y2="8.89" width="0.3048" layer="1"/>
 <wire x1="13.97" y1="10.16" x2="12.065" y2="10.16" width="0.3048" layer="1"/>
